Commit message: 3 19

File: legged_gym/resources/robots/g1/urdf/g1_29dof_rev_1_0_allcollision.urdf (robot description, URDF)
Before this commit: robot g1_29dof_rev_1_0, 47 links, 46 joints
Links:
- link left_elbow_link: geometry collision mesh filename=../meshes/left_elbow_link.STL; visual mesh filename=../meshes/left_elbow_link.STL
- link left_hip_roll_link: geometry collision mesh filename=../meshes/left_hip_roll_link.STL; visual mesh filename=../meshes/left_hip_roll_link.STL
- link left_hip_yaw_link: geometry collision mesh filename=../meshes/left_hip_yaw_link.STL; visual mesh filename=../meshes/left_hip_yaw_link.STL
- link left_shoulder_roll_link: geometry collision mesh filename=../meshes/left_shoulder_roll_link.STL; visual mesh filename=../meshes/left_shoulder_roll_link.STL
- link left_shoulder_yaw_link: geometry collision mesh filename=../meshes/left_shoulder_yaw_link.STL; visual mesh filename=../meshes/left_shoulder_yaw_link.STL
- link left_wrist_pitch_link: geometry collision mesh filename=../meshes/left_wrist_pitch_link.STL; visual mesh filename=../meshes/left_wrist_pitch_link.STL
- link left_wrist_roll_link: geometry collision mesh filename=../meshes/left_wrist_roll_link.STL; visual mesh filename=../meshes/left_wrist_roll_link.STL
- link left_wrist_yaw_link: geometry collision mesh filename=../meshes/left_wrist_yaw_link.STL; visual mesh filename=../meshes/left_wrist_yaw_link.STL
- link right_elbow_link: geometry collision mesh filename=../meshes/right_elbow_link.STL; visual mesh filename=../meshes/right_elbow_link.STL
- link right_hip_roll_link: geometry collision mesh filename=../meshes/right_hip_roll_link.STL; visual mesh filename=../meshes/right_hip_roll_link.STL
- link right_hip_yaw_link: geometry collision mesh filename=../meshes/right_hip_yaw_link.STL; visual mesh filename=../meshes/right_hip_yaw_link.STL
- link right_shoulder_roll_link: geometry collision mesh filename=../meshes/right_shoulder_roll_link.STL; visual mesh filename=../meshes/right_shoulder_roll_link.STL
- link right_shoulder_yaw_link: geometry collision mesh filename=../meshes/right_shoulder_yaw_link.STL; visual mesh filename=../meshes/right_shoulder_yaw_link.STL
- link right_wrist_pitch_link: geometry collision mesh filename=../meshes/right_wrist_pitch_link.STL; visual mesh filename=../meshes/right_wrist_pitch_link.STL
- link right_wrist_roll_link: geometry collision mesh filename=../meshes/right_wrist_roll_link.STL; visual mesh filename=../meshes/right_wrist_roll_link.STL
- link right_wrist_yaw_link: geometry collision mesh filename=../meshes/right_wrist_yaw_link.STL; visual mesh filename=../meshes/right_wrist_yaw_link.STL
- link torso_link: geometry collision mesh filename=../meshes/torso_link_rev_1_0.STL; visual mesh filename=../meshes/torso_link_rev_1_0.STL

Commit message: 3.22

File: legged_gym/resources/robots/g1/urdf/g1_29dof_rev_1_0_allcollision.urdf (robot description, URDF)
Before this commit: robot g1_29dof_rev_1_0, 47 links, 46 joints
Links:
- link left_hip_pitch_link: geometry collision mesh filename=../meshes/left_hip_pitch_link.STL; visual mesh filename=../meshes/left_hip_pitch_link.STL
- link logo_link: geometry collision mesh filename=../meshes/logo_link.STL; visual mesh filename=../meshes/logo_link.STL
- link pelvis_contour_link: geometry collision mesh filename=../meshes/pelvis_contour_link.STL; visual mesh filename=../meshes/pelvis_contour_link.STL
- link right_hip_pitch_link: geometry collision mesh filename=../meshes/right_hip_pitch_link.STL; visual mesh filename=../meshes/right_hip_pitch_link.STL
